File: _autosave-HL2_MRF101.kicad_pcb (KiCad board)
At the start: 4 copper layers, 149.9 x 100 mm, 190 parts, among them J1 Antenna, J2 HL2, J3 RF3, J4 RF1, J5 RCJ-041, J6 50VDC, J7 12V, J8 Fan, J9 HL2_12V, K1 EC2-3NU, K10 EC2-3NU, K11 EC2-3NU, K12 EC2-3NU, K13 EC2-3NU, K2 EC2-3NU, K3 EC2-3NU, K4 EC2-3NU, K5 EC2-3NU, K6 EC2-3NU, K7 EC2-3NU, K8 EC2-3NU, K9 EC2-3NU, Q1 MRF101AN, Q2 2N7002, Q3 NSS60601MZ4, T1 Coupler, T2 Coupler, T3 744851330, U1 MCP6282E/MS, U3 MCP23008, U4 ULN2003, U5 LM35-NEB, U6 LM393

Commit message: Revision 0.1 finished
Parts:
- added REF**: OSHW-Logo2_7.3x6mm_SilkScreen, Symbol:OSHW-Logo2_7.3x6mm_SilkScreen, B.Cu at (152.6, 134.2)
- added REF**: OSHW-Logo2_7.3x6mm_SilkScreen, Symbol:OSHW-Logo2_7.3x6mm_SilkScreen, F.Cu at (152.6, 134.2)
- added REF**: VAL**, n2adr:m3, F.Cu at (205.0, 137.0)
- added REF**: VAL**, n2adr:m3, F.Cu at (205.0, 43.0)
- Band 7: renamed from TP14
- moved C69 2.51 mm to (208.9, 124.1)
- moved C74 2.51 mm to (204.8, 124.1)
- moved C77 2.51 mm to (200.8, 124.1)
- moved L15 2.51 mm to (208.3, 127.8)
- moved L16 2.51 mm to (201.3, 127.8)
- moved TP4 1.40 mm to (154.2, 129.0)
- renumbered TP6 to CN8, TP7 to INTTR
Routing:
- net +3V3: track 362.7 -> 356.1 mm
- net Net-(C69-Pad2): track 40.1 -> 34.4 mm
- net GND: track 251.0 -> 248.6 mm, vias 200 -> 197
- net Net-(C77-Pad1): track 10.3 -> 9.44 mm
- net Net-(TP4-Pad1): track 19.5 -> 18.7 mm
Other:
- board text added: "Bias 100 mA"
- board text added: "MRF101 100W PA for Hermes-Lite 2 © 2020 DB9MAT - based on work by WA2EUJ and N2ADR"
