File: HL2_MRF101.sch (KiCad schematic (older format))
At the start: 168 parts, among them J1 Antenna, J2 HL2, J3 50VDC, J4 RF1, J5 RCJ-041, K1 EC2-3NU, K10 EC2-3NU, K11 EC2-3NU, K12 EC2-3NU, K13 EC2-3NU, K2 EC2-3NU, K3 EC2-3NU, K4 EC2-3NU, K5 EC2-3NU, K6 EC2-3NU, K7 EC2-3NU, K8 EC2-3NU, K9 EC2-3NU, Q1 MRF101AN, Q2 2N7002, T1 10t, T2 10t, T3 744851330, U1 MCP6282E/MS, U2 MCP23008, U3 ULN2003, U4 74LVC1G00

Commit message: Updated schematics; added footprints
Parts:
- removed C67: 330u, symbol Device:C_Small
- removed JP1, JP2: 1t, symbol Device:Jumper_NC_Small
- removed T1, T2: 10t, symbol Device:L
- added C67: 330u/ 63V, Capacitor_THT:CP_Radial_D10.0mm_P5.00mm, symbol Device:CP_Small
- added J3: RF3, n2adr:BNCEDGE, symbol Connector:Conn_Coaxial
- added R1: 100, Resistor_SMD:R_0805_2012Metric, symbol Device:R_Small
- added R12, R3: DNI, Resistor_SMD:R_0805_2012Metric, symbol Device:R_Small
- added R13, R16, R17, R2: 0, Resistor_SMD:R_0805_2012Metric, symbol Device:R_Small
- added T1, T2: Coupler, T50:T50_Coupler, symbol HL2-MRF101:Coupler
- added TP1: P8, TestPoint:TestPoint_Pad_D1.5mm, symbol Connector:TestPoint
- added TP2: GND, TestPoint:TestPoint_Pad_D1.5mm, symbol Connector:TestPoint
- C1, C2, C3, C37, C38, C39, C4, C40, C41, C42, C43, C44, C48, C49, C5, C50, C51, C52, C53, C62, C63, C64, C65, C66, C68, C69, C70, C71, C72, C73, C74, C75, C76, C77: footprint (none) -> Capacitor_SMD:C_0805_2012Metric
- C10, C11, C19, C20, C21, C22, C23, C24, C25, C26, C27, C28, C29, C30, C31, C32, C33, C34, C35, C36, C6, C7, C8, C9: footprint (none) -> Capacitor_SMD:C_1206_3216Metric
- C12: renamed from C13; footprint (none) -> Capacitor_SMD:C_1206_3216Metric
- C13: renamed from C14; footprint (none) -> Capacitor_SMD:C_1206_3216Metric
- C14: renamed from C15; footprint (none) -> Capacitor_SMD:C_1206_3216Metric
- C15: renamed from C16; footprint (none) -> Capacitor_SMD:C_1206_3216Metric
- C16: renamed from C17; footprint (none) -> Capacitor_SMD:C_1206_3216Metric
- C17: renamed from C18; footprint (none) -> Capacitor_SMD:C_1206_3216Metric
- C18: renamed from C12; footprint (none) -> Capacitor_SMD:C_0805_2012Metric
- C45: renamed from C46; footprint (none) -> Capacitor_SMD:C_0805_2012Metric
- C46: renamed from C47; footprint (none) -> Capacitor_SMD:C_0805_2012Metric
- C47: renamed from C45; footprint (none) -> Capacitor_SMD:C_0805_2012Metric
- C54: renamed from C55; footprint (none) -> Capacitor_SMD:C_0805_2012Metric
- C55: renamed from C56; footprint (none) -> Capacitor_SMD:C_0805_2012Metric
- C56: renamed from C57; footprint (none) -> Capacitor_SMD:C_0805_2012Metric
- C57: renamed from C58; footprint (none) -> Capacitor_SMD:C_0805_2012Metric
- C58: renamed from C59; footprint (none) -> Capacitor_SMD:C_0805_2012Metric
- C59: renamed from C60; footprint (none) -> Capacitor_SMD:C_0805_2012Metric
- C60: renamed from C61; footprint (none) -> Capacitor_SMD:C_0805_2012Metric
- C61: renamed from C54; footprint (none) -> Capacitor_SMD:CP_Elec_6.3x5.9
- D1, D2: footprint Diode_THT:D_DO-35_SOD27_P7.62mm_Horizontal -> Diode_SMD:D_SOD-123
- D3, D4: footprint (none) -> Diode_SMD:D_SOD-123
- FB1, FB2, FB3: footprint (none) -> Inductor_SMD:L_0805_2012Metric
- J1: footprint (none) -> TerminalBlock_Phoenix:TerminalBlock_Phoenix_PT-1,5-2-3.5-H_1x02_P3.50mm_Horizontal
- J2: footprint (none) -> Connector_PinHeader_2.54mm:PinHeader_1x20_P2.54mm_Vertical
- J4: footprint (none) -> n2adr:BNCEDGE
- J5: footprint (none) -> n2adr:PhonoRcaRCJ-04x
- J6: renamed from J3; footprint (none) -> TerminalBlock_Phoenix:TerminalBlock_Phoenix_PT-1,5-2-5.0-H_1x02_P5.00mm_Horizontal
- K1, K10, K11, K12, K13, K2, K3, K4, K5, K6, K7, K8, K9: footprint (none) -> n2adr:RelayDPDT01
- L1, L10, L11, L12, L2, L3, L4, L5, L6, L7, L8, L9: footprint (none) -> T50:T50_V_THT
- L13: renamed from L14; footprint (none) -> Inductor_SMD:L_0805_2012Metric
- L14: renamed from L13; footprint (none) -> n2adr:SignalCommunications-WE-PF_7427929XXX
- L15, L16: footprint (none) -> Inductor_SMD:L_1812_4532Metric
- Q1: footprint (none) -> Package_TO_SOT_THT:TO-220-3_Vertical
- R10: renamed from R7; footprint (none) -> Resistor_SMD:R_0805_2012Metric
- R11: renamed from R8; footprint (none) -> Resistor_SMD:R_0805_2012Metric
- R14: renamed from R15; footprint (none) -> Resistor_SMD:R_0805_2012Metric
- R15: renamed from R9; footprint (none) -> Resistor_SMD:R_0805_2012Metric
- R18: renamed from R10; footprint (none) -> Resistor_SMD:R_2512_6332Metric
- R19: renamed from R11; footprint (none) -> Resistor_SMD:R_2512_6332Metric
- R20: renamed from R12; footprint (none) -> Resistor_SMD:R_2512_6332Metric
- R21: renamed from R13; footprint (none) -> Resistor_SMD:R_2512_6332Metric
- R22: renamed from R14; footprint (none) -> Resistor_SMD:R_2512_6332Metric
- R23: renamed from R16; footprint (none) -> Resistor_SMD:R_2512_6332Metric
- R24: renamed from R17; footprint (none) -> Resistor_SMD:R_2512_6332Metric
- R25: renamed from R18; footprint (none) -> Resistor_SMD:R_2512_6332Metric
- R26: renamed from R19; footprint (none) -> Resistor_SMD:R_2512_6332Metric
- R27: renamed from R20; footprint (none) -> Resistor_SMD:R_2512_6332Metric
- R28: renamed from R21; footprint (none) -> Resistor_SMD:R_2512_6332Metric
- R29: renamed from R22; footprint (none) -> Resistor_SMD:R_0815_2038Metric
- R30: renamed from R23; footprint (none) -> Resistor_SMD:R_2512_6332Metric
- R31: renamed from R24; footprint (none) -> Resistor_SMD:R_0805_2012Metric
- R32: renamed from R25; footprint (none) -> Resistor_SMD:R_0805_2012Metric
- R4: renamed from R1; footprint (none) -> Resistor_SMD:R_0805_2012Metric
- R5: renamed from R2; footprint (none) -> Resistor_SMD:R_0805_2012Metric
- R6: renamed from R3; footprint (none) -> Resistor_SMD:R_0805_2012Metric
- R7: renamed from R4; footprint (none) -> Resistor_SMD:R_0805_2012Metric
- R8: renamed from R5; footprint (none) -> Resistor_SMD:R_0805_2012Metric
- R9: renamed from R6; footprint (none) -> Resistor_SMD:R_0805_2012Metric
- RV1: footprint (none) -> Potentiometer_THT:Potentiometer_Bourns_3386P_Vertical
- T3: footprint (none) -> n2adr:SignalCommunications-WE-DCT
- TP10: renamed from TP8; footprint (none) -> TestPoint:TestPoint_Pad_D1.5mm
- TP11: renamed from TP9; footprint (none) -> TestPoint:TestPoint_Pad_D1.5mm
- TP12: renamed from TP10; footprint (none) -> TestPoint:TestPoint_Pad_D1.5mm
- TP13: renamed from TP11; footprint (none) -> TestPoint:TestPoint_Pad_D1.5mm
- TP14: renamed from TP12; footprint (none) -> TestPoint:TestPoint_Pad_D1.5mm
- TP3: value RF3 -> P8; footprint (none) -> TestPoint:TestPoint_Pad_D1.5mm
- TP4: renamed from TP1; footprint (none) -> TestPoint:TestPoint_Pad_D1.5mm
- TP5: renamed from TP2; footprint (none) -> TestPoint:TestPoint_Pad_D1.5mm
- TP6: renamed from TP4; footprint (none) -> TestPoint:TestPoint_Pad_D1.5mm
- TP7: renamed from TP5; footprint (none) -> TestPoint:TestPoint_Pad_D1.5mm
- TP8: renamed from TP6; footprint (none) -> TestPoint:TestPoint_Pad_D1.5mm
- TP9: renamed from TP7; footprint (none) -> TestPoint:TestPoint_Pad_D1.5mm
- U1: footprint (none) -> Package_SO:MSOP-8_3x3mm_P0.65mm
- U2: renamed from U4; footprint (none) -> Package_TO_SOT_SMD:SOT-23-5
- U3: renamed from U2; footprint (none) -> Package_SO:SSOP-20_5.3x7.2mm_P0.65mm
- U4: renamed from U3; footprint (none) -> Package_SO:TSSOP-16_4.4x5mm_P0.65mm
Connections:
- wire segments 697 -> 712
Other:
- note added: "RF1: Low Power TX\nRF3: Optional RX, used for Pure Signal"
- moved on the sheet: J5

Commit message: Components layed out
Parts:
- removed C61: 10u / 63V, Capacitor_SMD:CP_Elec_6.3x5.9, symbol Device:CP_Small
- added C61: 1u, Capacitor_SMD:C_0805_2012Metric, symbol Device:C_Small
- added C78, C79: 100n, Capacitor_SMD:C_0805_2012Metric, symbol Device:C_Small
- added J7: 12V, TerminalBlock_Phoenix:TerminalBlock_Phoenix_PT-1,5-2-3.5-H_1x02_P3.50mm_Horizontal, symbol Connector_Generic:Conn_01x02
- added J8: Fan, Connector_JST:JST_XH_B2B-XH-A_1x02_P2.50mm_Vertical, symbol Connector_Generic:Conn_01x02
- added J9: HL2_12V, Connector_PinSocket_2.54mm:PinSocket_1x03_P2.54mm_Vertical, symbol Connector_Generic:Conn_01x03
- added Q3: NSS60601MZ4, Package_TO_SOT_SMD:SOT-223-3_TabPin2, symbol Device:Q_NPN_BCE
- added R33, R34, R36, R37: 10k, Resistor_SMD:R_0805_2012Metric, symbol Device:R_Small
- added R35: 560k, Resistor_SMD:R_0805_2012Metric, symbol Device:R_Small
- added RV2: 10k, Potentiometer_SMD:Potentiometer_Bourns_3314J_Vertical, symbol Device:R_POT_Small
- added U5: LM35-NEB, Package_TO_SOT_THT:TO-220-3_Vertical, symbol Sensor_Temperature:LM35-NEB
- added U6: LM393, Package_SO:SOP-8_3.76x4.96mm_P1.27mm, symbol Comparator:LM393
- R29: footprint Resistor_SMD:R_0815_2038Metric -> Resistor_SMD:R_0805_2012Metric
- RV1: footprint Potentiometer_THT:Potentiometer_Bourns_3386P_Vertical -> Potentiometer_SMD:Potentiometer_Bourns_3314J_Vertical
Connections:
- net labels added: +12V
- net labels removed: +48V
- wire segments 712 -> 759

Commit message: Revision 0.1 finished
Parts:
- removed R14: 10k, Resistor_SMD:R_0805_2012Metric, symbol Device:R_Small
- removed TP13: P8, TestPoint:TestPoint_Pad_D1.5mm, symbol Connector:TestPoint
- removed U2: 74LVC1G00, Package_TO_SOT_SMD:SOT-23-5, symbol 74xGxx:74LVC1G00
- C10, C35: value 180p -> 560p
- C11, C36: value 100p -> 1200p
- C12, C25: value 470p -> 39p
- C13, C26: value 220p -> 56p
- C14, C27: value 150p -> 120p
- C15, C28: value 120p -> 150p
- C16, C29: value 56p -> 220p
- C17, C30: value 39p -> 470p
- C19: value 2200p -> 180p
- C20: value 1200p -> 330p
- C21: value 1000p -> 680p
- C22: value 680p -> 1000p
- C23: value 330p -> 1200p
- C24: value 180p -> 2200p
- C31, C6: value 1200p -> 100p
- C32, C7: value 560p -> 180p
- C33, C8: value 560p -> 390p
- C34, C9: value 390p -> 560p
- L1, L7: value 3.1u -> 224n
- L10, L4: value 680n -> 1.1u
- L11, L5: value 385n -> 1.7u
- L12, L6: value 224n -> 3.1u
- L2, L8: value 1.7u -> 385n
- L3, L9: value 1.1u -> 680n
Connections:
- net labels removed: BIAS_ON, PTT
- wire segments 759 -> 750
- no-connect marks 1 -> 3
Other:
- note added: "0V: Bias On\n3V: Bias Off"
- note added: "20 dB Coupler\nFT50A-61\n1 Turn #18 Teflon\n10 Turn #28 Enameled"
- note removed: "20 dB Coupler\nFT50-61\n1 Turn #18 Teflon\n10 Turn #28 Enameled"
- note removed: "3V: Bias On\n0V: Bias Off"
- note removed: "BIAS_ON: GND on Rx, +3.3V on Tx"

Commit message: Updated R6-9 to 1206 1/2W
Parts:
- J1: footprint TerminalBlock_Phoenix:TerminalBlock_Phoenix_PT-1,5-2-3.5-H_1x02_P3.50mm_Horizontal -> Connector_Coaxial:BNC_Amphenol_B6252HB-NPP3G-50_Horizontal
- J2: footprint Connector_PinHeader_2.54mm:PinHeader_1x20_P2.54mm_Vertical -> Connector_PinSocket_2.54mm:PinSocket_1x20_P2.54mm_Vertical
- R6, R7, R8, R9: footprint Resistor_SMD:R_0805_2012Metric -> Resistor_SMD:R_1206_3216Metric
Changed lines of the file:
@@
 F 0 "J1" H 5350 8925 50  0000 L CNN
 F 1 "Antenna" H 5350 8834 50  0000 L CNN
-F 2 "TerminalBlock_Phoenix:TerminalBlock_Phoenix_PT-1,5-2-3.5-H_1x02_P3.50mm_Horizontal" H 5250 8950 50  0001 C CNN
+F 2 "Connector_Coaxial:BNC_Amphenol_B6252HB-NPP3G-50_Horizontal" H 5250 8950 50  0001 C CNN
 F 3 " ~" H 5250 8950 50  0001 C CNN
 	1    5250 8950
@@
 F 0 "R9" H 4859 10246 50  0000 L CNN
 F 1 "100" H 4859 10155 50  0000 L CNN
-F 2 "Resistor_SMD:R_0805_2012Metric" H 4800 10200 50  0001 C CNN
+F 2 "Resistor_SMD:R_1206_3216Metric" H 4800 10200 50  0001 C CNN
 F 3 "~" H 4800 10200 50  0001 C CNN
 	1    4800 10200
@@
 F 0 "R8" H 4542 10154 50  0000 R CNN
 F 1 "100" H 4542 10245 50  0000 R CNN
-F 2 "Resistor_SMD:R_0805_2012Metric" H 4600 10200 50  0001 C CNN
+F 2 "Resistor_SMD:R_1206_3216Metric" H 4600 10200 50  0001 C CNN
 F 3 "~" H 4600 10200 50  0001 C CNN
 	1    4600 10200
@@
 F 0 "R7" H 4109 10246 50  0000 L CNN
 F 1 "100" H 4109 10155 50  0000 L CNN
-F 2 "Resistor_SMD:R_0805_2012Metric" H 4050 10200 50  0001 C CNN
+F 2 "Resistor_SMD:R_1206_3216Metric" H 4050 10200 50  0001 C CNN
 F 3 "~" H 4050 10200 50  0001 C CNN
 	1    4050 10200
@@
 F 0 "R6" H 3792 10154 50  0000 R CNN
 F 1 "100" H 3792 10245 50  0000 R CNN
-F 2 "Resistor_SMD:R_0805_2012Metric" H 3850 10200 50  0001 C CNN
+F 2 "Resistor_SMD:R_1206_3216Metric" H 3850 10200 50  0001 C CNN
 F 3 "~" H 3850 10200 50  0001 C CNN
 	1    3850 10200
@@
 F 0 "J2" H 8268 8675 50  0000 C CNN
 F 1 "HL2" H 8268 8766 50  0000 C CNN
-F 2 "Connector_PinHeader_2.54mm:PinHeader_1x20_P2.54mm_Vertical" H 8350 9900 50  0001 C CNN
+F 2 "Connector_PinSocket_2.54mm:PinSocket_1x20_P2.54mm_Vertical" H 8350 9900 50  0001 C CNN
 F 3 "~" H 8350 9900 50  0001 C CNN
 	1    8350 9900

Commit message: Reworked Op Amps
Parts:
- removed RV2: 10k, Potentiometer_SMD:Potentiometer_Bourns_3314J_Vertical, symbol Device:R_POT_Small
- removed U6: LM393, Package_SO:SOP-8_3.76x4.96mm_P1.27mm, symbol Comparator:LM393
- added R?: 10k, Resistor_SMD:R_0805_2012Metric, symbol Device:R_Small
- added R?: 12k, Resistor_SMD:R_0805_2012Metric, symbol Device:R_Small
- added U? (x2): MCP6282E/MS, Package_SO:MSOP-8_3x3mm_P0.65mm, symbol Device:Opamp_Dual_Generic
- R10, R5: value 100k -> 56k
- R34: value 10k -> 62k
- R35: value 560k -> 220k
- R6, R7, R8, R9: footprint Resistor_SMD:R_1206_3216Metric -> Resistor_SMD:R_2512_6332Metric
Connections:
- wire segments 750 -> 746
Other:
- note added: "10mV/°C\n55°C => 550mV\n40°C => 400mV"
- note removed: "Todo: check voltages/amplification"

Commit message: Updated layout
Parts:
- C1, C10, C11, C12, C13, C14, C15, C16, C17, C18, C19, C2, C20, C21, C22, C23, C24, C25, C26, C27, C28, C29, C3, C30, C31, C32, C33, C34, C35, C36, C37, C38, C39, C4, C40, C41, C42, C43, C44, C45, C46, C47, C48, C49, C5, C50, C51, C52, C53, C54, C55, C56, C57, C58, C59, C6, C60, C61, C62, C63, C64, C65, C66, C68, C69, C7, C70, C71, C72, C73, C74, C75, C76, C77, C78, C79, C8, C9: symbol Device:C_Small -> HL2_MRF101-rescue:C_Small-Device
- C67: symbol Device:CP_Small -> HL2_MRF101-rescue:CP_Small-Device
- D1, D2: symbol Diode:1N5711 -> HL2_MRF101-rescue:1N5711-Diode
- D3: symbol Device:D_Small -> HL2_MRF101-rescue:D_Small-Device
- D4: symbol Device:D_Zener -> HL2_MRF101-rescue:D_Zener-Device
- D5: symbol Diode:1N4148 -> HL2_MRF101-rescue:1N4148-Diode
- FB1, FB2, FB3: symbol Device:Ferrite_Bead_Small -> HL2_MRF101-rescue:Ferrite_Bead_Small-Device
- J1, J3, J4: symbol Connector:Conn_Coaxial -> HL2_MRF101-rescue:Conn_Coaxial-Connector
- J2: symbol Connector_Generic:Conn_01x20 -> HL2_MRF101-rescue:Conn_01x20-Connector_Generic
- J6, J7, J8: symbol Connector_Generic:Conn_01x02 -> HL2_MRF101-rescue:Conn_01x02-Connector_Generic
- J9: symbol Connector_Generic:Conn_01x03 -> HL2_MRF101-rescue:Conn_01x03-Connector_Generic
- L1, L10, L11, L12, L13, L14, L15, L16, L2, L3, L4, L5, L6, L7, L8, L9: symbol Device:L_Small -> HL2_MRF101-rescue:L_Small-Device
- Q1: symbol Device:Q_NMOS_GSD -> HL2_MRF101-rescue:Q_NMOS_GSD-Device
- Q2: symbol Transistor_FET:2N7002 -> HL2_MRF101-rescue:2N7002-Transistor_FET
- Q3: symbol Device:Q_NPN_BCE -> HL2_MRF101-rescue:Q_NPN_BCE-Device
- R1, R10, R11, R12, R13, R15, R16, R17, R18, R19, R2, R20, R21, R22, R23, R24, R25, R26, R27, R28, R29, R3, R30, R31, R32, R33, R34, R35, R36, R37, R4, R5, R6, R7, R8, R9: symbol Device:R_Small -> HL2_MRF101-rescue:R_Small-Device
- R14, R38: renamed from R?; symbol Device:R_Small -> HL2_MRF101-rescue:R_Small-Device
- RV1: symbol Device:R_POT -> HL2_MRF101-rescue:R_POT-Device
- TP1, TP10, TP11, TP12, TP14, TP2, TP3, TP4, TP5, TP6, TP7, TP8, TP9: symbol Connector:TestPoint -> HL2_MRF101-rescue:TestPoint-Connector
- U1: symbol Device:Opamp_Dual_Generic -> HL2_MRF101-rescue:Opamp_Dual_Generic-Device
- U2: renamed from U?; symbol Device:Opamp_Dual_Generic -> HL2_MRF101-rescue:Opamp_Dual_Generic-Device
- U4: symbol Transistor_Array:ULN2003 -> HL2_MRF101-rescue:ULN2003-Transistor_Array
- U5: symbol Sensor_Temperature:LM35-NEB -> HL2_MRF101-rescue:LM35-NEB-Sensor_Temperature

Commit message: Started adding current monitor
Parts:
- added U?: INA193, Package_TO_SOT_SMD:SOT-23-5, symbol Amplifier_Current:INA193
Other:
- note added: "Based on WA2EUJ MRF101 EVB and N2ADR Filter Board\nhttps://rfpowertools.com http://james.ahlstrom.name/hl2filter/"
- note removed: "Based on WA2EUJ MRF101 EVB\nhttps://rfpowertools.com\n\nand\n\nN2ADR Filter Board\nhttp://james.ahlstrom.name/hl2filter/"
- moved on the sheet: C47, C54, C55, C57, C58, C61, C64, C65, C68, C69, C73, C74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

Commit message: Added bias control and current monitor
Parts:
- removed R14, R36: 10k, Resistor_SMD:R_0805_2012Metric, symbol HL2_MRF101-rescue:R_Small-Device
- removed R34: 62k, Resistor_SMD:R_0805_2012Metric, symbol HL2_MRF101-rescue:R_Small-Device
- removed R35: 220k, Resistor_SMD:R_0805_2012Metric, symbol HL2_MRF101-rescue:R_Small-Device
- removed R38: 12k, Resistor_SMD:R_0805_2012Metric, symbol HL2_MRF101-rescue:R_Small-Device
- removed RV1: 10k, Potentiometer_SMD:Potentiometer_Bourns_3314J_Vertical, symbol HL2_MRF101-rescue:R_POT-Device
- removed TP2: GND, TestPoint:TestPoint_Pad_D1.5mm, symbol HL2_MRF101-rescue:TestPoint-Connector
- removed U2: MCP6282E/MS, Package_SO:MSOP-8_3x3mm_P0.65mm, symbol HL2_MRF101-rescue:Opamp_Dual_Generic-Device
- added C80: 4n7, Capacitor_SMD:C_0805_2012Metric, symbol HL2_MRF101-rescue:C_Small-Device
- added C81, C82: 100n, Capacitor_SMD:C_0805_2012Metric, symbol HL2_MRF101-rescue:C_Small-Device
- added C83: DNI, symbol device:C_Small
- added FB4, FB5, FB6, FB7, FB8: FB, symbol device:Ferrite_Bead_Small
- added R14, R35: DNI, symbol device:R_Small
- added R34: 0.036, symbol device:R_Shunt
- added U2: MAX11613, MODULE, symbol hermeslite:MAX11613
- added U6: MCP4561, symbol HL2-MRF101:MCP4561
- C79: value 100n -> 4n7
- U7: renamed from U?; symbol Amplifier_Current:INA193 -> HL2_MRF101-rescue:INA193-Amplifier_Current
Connections:
- net +3V3: now also FB4.1, FB5.1, FB6.2, FB7.2, FB8.2; no longer C47.2, C54.2, C55.2, C79.1, U1.8 (V+)
- net GND: now also C78.1, C79.1, U7.2 (GND), C80.1, C81.2, C82.2, U2.7 (GND), U6.1 (A0), U6.4 (Vss); no longer C78.2, C79.2
- net SCL: now also U2.5 (SCL), U6.2 (SCL)
- net SDA: now also U2.6 (SDA), U6.3 (SDA)
- net at C63.2, D4.1 (K), Q2.3 (D)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: now also U6.5 (P0A)
- net at C59.1, R26.2: now also U6.6 (P0W)
- net at R29.1: now also U6.7 (P0B)
- net at C67.1, C70.2, C71.2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: now also R34.4; no longer L14.2, R32.1
- net Vipa: now reaches U7.1
- net Vipa: now also C79.2, U2.2 (AIN1)
- net at U7.3 (+): now also C83.1, R14.1
- net at U7.4 (-): now also C83.2, R35.1
- net at U7.5 (V+): now also C81.1, FB6.1
- net Vtemp: now reaches R33.1, U5.3 (Vout)
- net Vtemp: now also C80.2, U2.1 (AIN0)
- net Fan_PWM: now reaches Q3.1 (B), R37.2
- new net: L14.2, R32.1, R34.1
- new net: R14.2, R34.2
- new net: R34.3, R35.2
- new net: C47.2, FB8.1, U1.8 (V+)
- new net: C78.2, FB4.2, U2.8 (Vdd)
- new net: C54.2, C55.2, FB5.2
- new net: C82.1, FB7.1, U6.8 (Vdd)
- no-connect marks 3 -> 5
Other:
- note added: "4A => 144mV"
- note added: "Gain 20V/V\n4A => 2.88V"
- note added: "I2C Addr 0x2E"
- note added: "I2C Addr. 0x20"
- note added: "I2C Addr. 0x34"
- note added: "set for 100mA\n=> Vipa = 72mV"
- note removed: "set for 100mA"
- moved on the sheet: C18, C37, C47, C54, C55, C56, C57, C58, C59, C60, C61, C62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
