File: HL2_MRF101.sch (KiCad schematic (older format))
At the start: 195 parts, among them J1 Antenna, J2 HL2, J3 RF3, J4 RF1, J5 RCJ-041, J6 50VDC, J7 12V, J8 Fan, J9 HL2_12V, K1 EC2-3NU, K10 EC2-3NU, K11 EC2-3NU, K12 EC2-3NU, K13 EC2-3NU, K2 EC2-3NU, K3 EC2-3NU, K4 EC2-3NU, K5 EC2-3NU, K6 EC2-3NU, K7 EC2-3NU, K8 EC2-3NU, K9 EC2-3NU, Q1 MRF101AN, Q2 2N7002, Q3 NSS60601MZ4, T1 Coupler, T2 Coupler, T3 744851330, U1 MCP6282E/MS, U2 MAX11613, U3 MCP23008, U4 ULN2003, U5 LM35-NEB, U6 MCP4561, U7 INA193

Commit message: Started current monitor layout
Parts:
- removed R34: 0.036, symbol device:R_Shunt
- removed TP4: P8, TestPoint:TestPoint_Pad_D1.5mm, symbol HL2_MRF101-rescue:TestPoint-Connector
- added R34: 0.036, Resistors_SMD:R_0612, symbol device:R_Small
- C78, C79, C80, C81, C82: footprint Capacitor_SMD:C_0805_2012Metric -> Capacitors_SMD:C_0805
- C83: footprint (none) -> Capacitors_SMD:C_0805
- FB4, FB5, FB6, FB7, FB8: footprint (none) -> Inductors_SMD:L_0805
- R14, R35: value DNI -> JNC; footprint (none) -> Resistors_SMD:R_0805
- U2: footprint MODULE -> n2adr:MAX11613
- U6: footprint (none) -> Housings_SSOP:MSOP-8_3x3mm_Pitch0.65mm
- U7: footprint Package_TO_SOT_SMD:SOT-23-5 -> TO_SOT_Packages_SMD:SOT-23-5
Connections:
- net labels added: Fan_Ctrl
- net labels removed: Fan_PWM
- wire segments 771 -> 773
Other:
- note added: "Set to 10k\nSet for 100mA\n=> Vipa = 72mV"
- note removed: "set for 100mA\n=> Vipa = 72mV"
Changed lines of the file:
@@
 Wire Wire Line
 	13900 4650 14000 4650
-Text Notes 9850 4700 0    50   ~ 0
-set for 100mA\n=> Vipa = 72mV
+Text Notes 9850 4800 0    50   ~ 0
+Set to 10k\nSet for 100mA\n=> Vipa = 72mV
 Text Notes 10100 6100 0    50   ~ 0
 1-2W max!
@@
 	8150 1400 8250 1400
 $Comp
-L power:+3.3V #PWR061
-U 1 1 61C43041
-P 8250 1250
-F 0 "#PWR061" H 8250 1100 50  0001 C CNN
-F 1 "+3.3V" H 8265 1423 50  0000 C CNN
-F 2 "" H 8250 1250 50  0001 C CNN
-F 3 "" H 8250 1250 50  0001 C CNN
-	1    8250 1250
-	1    0    0    -1
-$EndComp
-Wire Wire Line
-	8250 1250 8250 1400
-$Comp
-L HL2_MRF101-rescue:TestPoint-Connector TP4
-U 1 1 61D36C9F
-P 8450 1400
-F 0 "TP4" H 8508 1472 50  0000 L CNN
-F 1 "P8" V 8495 1588 50  0001 L CNN
-F 2 "TestPoint:TestPoint_Pad_D1.5mm" H 8650 1400 50  0001 C CNN
-F 3 "~" H 8650 1400 50  0001 C CNN
-	1    8450 1400
-	1    0    0    -1
-$EndComp
-Wire Wire Line
-	8150 1500 8450 1500
-$Comp
 L HL2_MRF101-rescue:ULN2003-Transistor_Array U4
 U 1 1 61DB578D
@@
 Wire Wire Line
 	8150 1700 8700 1700
-$Comp
-L power:+3.3V #PWR073
-U 1 1 6257E7BA
-P 10100 1250
-F 0 "#PWR073" H 10100 1100 50  0001 C CNN
-F 1 "+3.3V" H 10115 1423 50  0000 C CNN
-F 2 "" H 10100 1250 50  0001 C CNN
-F 3 "" H 10100 1250 50  0001 C CNN
-	1    10100 1250
-	1    0    0    -1
-$EndComp
-Wire Wire Line
-	10000 1400 10100 1400
-Wire Wire Line
-	10100 1250 10100 1400
 Wire Wire Line
 	7050 2200 7050 2500
@@
 F 0 "U7" H 15300 4050 50  0000 L CNN
 F 1 "INA193" H 15300 3950 50  0000 L CNN
-F 2 "Package_TO_SOT_SMD:SOT-23-5" H 15300 4250 50  0001 C CNN
+F 2 "TO_SOT_Packages_SMD:SOT-23-5" H 15300 4250 50  0001 C CNN
 F 3 "http://www.ti.com/lit/ds/symlink/ina193.pdf" H 15300 4250 50  0001 C CNN
 	1    15300 4250
 	1    0    0    -1
 $EndComp
-$Comp
-L device:R_Shunt R34
-U 1 1 5E275DCC
-P 14000 4250
-F 0 "R34" H 13912 4296 50  0000 R CNN
-F 1 "0.036" H 13912 4205 50  0000 R CNN
-F 2 "" V 13930 4250 50  0001 C CNN
-F 3 "~" H 14000 4250 50  0001 C CNN
-	1    14000 4250
-	1    0    0    -1
-$EndComp
 Wire Wire Line
 	13550 3950 14000 3950
-Wire Wire Line
-	14000 3950 14000 4050
 Connection ~ 14000 3950
 Wire Wire Line
-	14000 4450 14000 4650
-Wire Wire Line
 	14000 3950 14000 3000
 Wire Wire Line
@@
 P 14350 4150
 F 0 "R14" V 14250 4150 50  0000 C CNN
-F 1 "DNI" V 14350 4150 39  0000 C CNN
-F 2 "" H 14350 4150 50  0001 C CNN
+F 1 "JNC" V 14350 4150 39  0000 C CNN
+F 2 "Resistors_SMD:R_0805" H 14350 4150 50  0001 C CNN
 F 3 "~" H 14350 4150 50  0001 C CNN
 	1    14350 4150
@@
 P 14350 4350
 F 0 "R35" V 14250 4350 50  0000 C CNN
-F 1 "DNI" V 14350 4350 39  0000 C CNN
-F 2 "" H 14350 4350 50  0001 C CNN
+F 1 "JNC" V 14350 4350 39  0000 C CNN
+F 2 "Resistors_SMD:R_0805" H 14350 4350 50  0001 C CNN
 F 3 "~" H 14350 4350 50  0001 C CNN
 	1    14350 4350
 	0    1    1    0
 $EndComp
-Wire Wire Line
-	14150 4350 14250 4350
-Wire Wire Line
-	14150 4150 14250 4150
 $Comp
 L device:C_Small C83
@@
 F 0 "C83" H 14692 4296 50  0000 L CNN
 F 1 "DNI" H 14692 4205 50  0000 L CNN
-F 2 "" H 14600 4250 50  0001 C CNN
+F 2 "Capacitors_SMD:C_0805" H 14600 4250 50  0001 C CNN
 F 3 "~" H 14600 4250 50  0001 C CNN
 	1    14600 4250
@@
 F 0 "C81" H 15492 3746 50  0000 L CNN
 F 1 "100n" H 15492 3655 50  0000 L CNN
-F 2 "Capacitor_SMD:C_0805_2012Metric" H 15400 3700 50  0001 C CNN
+F 2 "Capacitors_SMD:C_0805" H 15400 3700 50  0001 C CNN
 F 3 "~" H 15400 3700 50  0001 C CNN
 	1    15400 3700
@@
 Connection ~ 15200 3700
 Wire Wire Line
-	8450 1400 8450 1500
-Wire Wire Line
 	8700 1400 8700 1700
 Wire Wire Line
@@
 F 0 "U2" H 14700 1187 50  0000 C CNN
 F 1 "MAX11613" H 14700 1278 49  0000 C CNN
-F 2 "MODULE" H 14700 1125 50  0001 C CNN
+F 2 "n2adr:MAX11613" H 14700 1125 50  0001 C CNN
 F 3 "DOCUMENTATION" H 14700 1300 50  0001 C CNN
 	1    14700 1600
@@
 F 0 "C78" H 15458 1804 50  0000 R CNN
 F 1 "100n" H 15458 1895 50  0000 R CNN
-F 2 "Capacitor_SMD:C_0805_2012Metric" H 15550 1850 50  0001 C CNN
+F 2 "Capacitors_SMD:C_0805" H 15550 1850 50  0001 C CNN
 F 3 "~" H 15550 1850 50  0001 C CNN
 	1    15550 1850
@@
 F 0 "FB4" H 15650 1296 50  0000 L CNN
 F 1 "FB" H 15650 1205 50  0000 L CNN
-F 2 "" V 15480 1250 50  0001 C CNN
+F 2 "Inductors_SMD:L_0805" V 15480 1250 50  0001 C CNN
 F 3 "~" H 15550 1250 50  0001 C CNN
 	1    15550 1250
@@
 F 0 "C79" H 13608 1904 50  0000 R CNN
 F 1 "4n7" H 13608 1995 50  0000 R CNN
-F 2 "Capacitor_SMD:C_0805_2012Metric" H 13700 1950 50  0001 C CNN
+F 2 "Capacitors_SMD:C_0805" H 13700 1950 50  0001 C CNN
 F 3 "~" H 13700 1950 50  0001 C CNN
 	1    13700 1950
@@
 F 0 "C80" H 14108 1904 50  0000 R CNN
 F 1 "4n7" H 14108 1995 50  0000 R CNN
-F 2 "Capacitor_SMD:C_0805_2012Metric" H 14200 1950 50  0001 C CNN
+F 2 "Capacitors_SMD:C_0805" H 14200 1950 50  0001 C CNN
 F 3 "~" H 14200 1950 50  0001 C CNN
 	1    14200 1950
@@
 Connection ~ 8550 10450
 Text GLabel 8450 10450 0    50   Input ~ 0
-Fan_PWM
+Fan_Ctrl
 Text GLabel 10750 10250 2    50   Input ~ 0
 Vtemp
@@
 F 0 "FB6" H 15100 3454 50  0000 R CNN
 F 1 "FB" H 15100 3545 50  0000 R CNN
-F 2 "" V 15130 3500 50  0001 C CNN
+F 2 "Inductors_SMD:L_0805" V 15130 3500 50  0001 C CNN
 F 3 "~" H 15200 3500 50  0001 C CNN
 	1    15200 3500
@@
 F 0 "FB8" H 15300 7804 50  0000 R CNN
 F 1 "FB" H 15300 7895 50  0000 R CNN
-F 2 "" V 15330 7850 50  0001 C CNN
+F 2 "Inductors_SMD:L_0805" V 15330 7850 50  0001 C CNN
 F 3 "~" H 15400 7850 50  0001 C CNN
 	1    15400 7850
@@
 F 0 "FB5" H 12050 1496 50  0000 L CNN
 F 1 "FB" H 12050 1405 50  0000 L CNN
-F 2 "" V 11880 1450 50  0001 C CNN
+F 2 "Inductors_SMD:L_0805" V 11880 1450 50  0001 C CNN
 F 3 "~" H 11950 1450 50  0001 C CNN
 	1    11950 1450
@@
 F 0 "U6" H 10150 4615 50  0000 C CNN
 F 1 "MCP4561" H 10150 4524 50  0000 C CNN
-F 2 "" H 9950 5700 50  0001 C CNN
+F 2 "Housings_SSOP:MSOP-8_3x3mm_Pitch0.65mm" H 9950 5700 50  0001 C CNN
 F 3 "" H 9950 5700 50  0001 C CNN
 	1    10150 4050
@@
 F 0 "C82" H 9342 3996 50  0000 L CNN
 F 1 "100n" H 9342 3905 50  0000 L CNN
-F 2 "Capacitor_SMD:C_0805_2012Metric" H 9250 3950 50  0001 C CNN
+F 2 "Capacitors_SMD:C_0805" H 9250 3950 50  0001 C CNN
 F 3 "~" H 9250 3950 50  0001 C CNN
 	1    9250 3950
@@
 F 0 "FB7" H 9150 3504 50  0000 R CNN
 F 1 "FB" H 9150 3595 50  0000 R CNN
-F 2 "" V 9180 3550 50  0001 C CNN
+F 2 "Inductors_SMD:L_0805" V 9180 3550 50  0001 C CNN
 F 3 "~" H 9250 3550 50  0001 C CNN
 	1    9250 3550
@@
 Text Notes 15300 4750 0    50   ~ 0
 Gain 20V/V\n4A => 2.88V
+$Comp
+L device:R_Small R34
+U 1 1 6355C858
+P 14000 4250
+F 0 "R34" H 13941 4204 50  0000 R CNN
+F 1 "0.036" H 13941 4295 50  0000 R CNN
+F 2 "Resistors_SMD:R_0612" H 14000 4250 50  0001 C CNN
+F 3 "~" H 14000 4250 50  0001 C CNN
+	1    14000 4250
+	1    0    0    1
+$EndComp
+Wire Wire Line
+	14000 4150 14250 4150
+Wire Wire Line
+	14000 4350 14250 4350
+Wire Wire Line
+	14000 4350 14000 4650
+Connection ~ 14000 4350
+Wire Wire Line
+	14000 3950 14000 4150
+Connection ~ 14000 4150
+Text GLabel 8250 1500 2    50   Input ~ 0
+Fan_Ctrl
+Wire Wire Line
+	8150 1500 8250 1500
+Wire Wire Line
+	11550 1400 11550 1650
+Wire Wire Line
+	10000 1400 10100 1400
+Connection ~ 11550 1650
+Wire Wire Line
+	8250 950  10100 950
+Wire Wire Line
+	10100 950  10100 1400
+Wire Wire Line
+	8250 950  8250 1400
+Connection ~ 10100 1400
+Wire Wire Line
+	10100 1400 11550 1400
 $EndSCHEMATC

Commit message: Further routing
Parts:
- C83: symbol device:C_Small -> HL2_MRF101-rescue:C_Small-device
- FB4, FB5, FB6, FB7, FB8: symbol device:Ferrite_Bead_Small -> HL2_MRF101-rescue:Ferrite_Bead_Small-device
- R14, R34, R35: symbol device:R_Small -> HL2_MRF101-rescue:R_Small-device
Connections:
- net at L14.2, R14.2, R34.2: no longer R32.1
- net at C67.1, C70.2, C71.2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: now also R32.1
Other:
- moved on the sheet: C81, C83, FB6, J6, L14, R14, R34, R35, U7
Changed lines of the file:
@@
 	8000 8300 8100 8300
 Wire Wire Line
-	14450 3100 14450 3400
+	14450 2850 14450 3150
 $Comp
 L power:GND #PWR080
 U 1 1 63EC0114
-P 14450 3400
-F 0 "#PWR080" H 14450 3150 50  0001 C CNN
-F 1 "GND" H 14455 3227 50  0000 C CNN
-F 2 "" H 14450 3400 50  0001 C CNN
-F 3 "" H 14450 3400 50  0001 C CNN
-	1    14450 3400
-	-1   0    0    -1
-$EndComp
-Wire Wire Line
-	14550 3100 14450 3100
-Wire Wire Line
-	14550 3000 14300 3000
+P 14450 3150
+F 0 "#PWR080" H 14450 2900 50  0001 C CNN
+F 1 "GND" H 14455 2977 50  0000 C CNN
+F 2 "" H 14450 3150 50  0001 C CNN
+F 3 "" H 14450 3150 50  0001 C CNN
+	1    14450 3150
+	-1   0    0    -1
+$EndComp
+Wire Wire Line
+	14550 2850 14450 2850
+Wire Wire Line
+	14550 2750 14300 2750
 $Comp
 L HL2_MRF101-rescue:L_Small-Device L14
 U 1 1 63DACD97
-P 14200 3000
-F 0 "L14" V 14385 3000 50  0000 C CNN
-F 1 "7427929112" V 14294 3000 50  0000 C CNN
-F 2 "n2adr:SignalCommunications-WE-PF_7427929XXX" H 14200 3000 50  0001 C CNN
-F 3 "~" H 14200 3000 50  0001 C CNN
-	1    14200 3000
+P 14200 2750
+F 0 "L14" V 14385 2750 50  0000 C CNN
+F 1 "7427929112" V 14294 2750 50  0000 C CNN
+F 2 "n2adr:SignalCommunications-WE-PF_7427929XXX" H 14200 2750 50  0001 C CNN
+F 3 "~" H 14200 2750 50  0001 C CNN
+	1    14200 2750
 	0    1    -1   0
 $EndComp
@@
 L HL2_MRF101-rescue:Conn_01x02-Connector_Generic J6
 U 1 1 63DAB1DA
-P 14750 3000
-F 0 "J6" H 14668 3217 50  0000 C CNN
-F 1 "50VDC" H 14668 3126 50  0000 C CNN
-F 2 "TerminalBlock_Phoenix:TerminalBlock_Phoenix_PT-1,5-2-5.0-H_1x02_P5.00mm_Horizontal" H 14750 3000 50  0001 C CNN
-F 3 "~" H 14750 3000 50  0001 C CNN
-	1    14750 3000
+P 14750 2750
+F 0 "J6" H 14668 2967 50  0000 C CNN
+F 1 "50VDC" H 14668 2876 50  0000 C CNN
+F 2 "TerminalBlock_Phoenix:TerminalBlock_Phoenix_PT-1,5-2-5.0-H_1x02_P5.00mm_Horizontal" H 14750 2750 50  0001 C CNN
+F 3 "~" H 14750 2750 50  0001 C CNN
+	1    14750 2750
 	1    0    0    -1
 $EndComp
@@
 L HL2_MRF101-rescue:INA193-Amplifier_Current U7
 U 1 1 5E683490
-P 15300 4250
-F 0 "U7" H 15300 4050 50  0000 L CNN
-F 1 "INA193" H 15300 3950 50  0000 L CNN
-F 2 "TO_SOT_Packages_SMD:SOT-23-5" H 15300 4250 50  0001 C CNN
-F 3 "http://www.ti.com/lit/ds/symlink/ina193.pdf" H 15300 4250 50  0001 C CNN
-	1    15300 4250
-	1    0    0    -1
-$EndComp
-Wire Wire Line
-	13550 3950 14000 3950
-Connection ~ 14000 3950
-Wire Wire Line
-	14000 3950 14000 3000
-Wire Wire Line
-	14000 3000 14100 3000
+P 15300 3700
+F 0 "U7" H 15300 3500 50  0000 L CNN
+F 1 "INA193" H 15300 3400 50  0000 L CNN
+F 2 "TO_SOT_Packages_SMD:SOT-23-5" H 15300 3700 50  0001 C CNN
+F 3 "http://www.ti.com/lit/ds/symlink/ina193.pdf" H 15300 3700 50  0001 C CNN
+	1    15300 3700
+	1    0    0    -1
+$EndComp
+Wire Wire Line
+	14000 2750 14100 2750
 $Comp
 L power:GND #PWR0113
 U 1 1 5E88B411
-P 15200 4650
-F 0 "#PWR0113" H 15200 4400 50  0001 C CNN
-F 1 "GND" H 15205 4477 50  0000 C CNN
-F 2 "" H 15200 4650 50  0001 C CNN
-F 3 "" H 15200 4650 50  0001 C CNN
-	1    15200 4650
-	-1   0    0    -1
-$EndComp
-Wire Wire Line
-	15200 4550 15200 4650
+P 15200 4100
+F 0 "#PWR0113" H 15200 3850 50  0001 C CNN
+F 1 "GND" H 15205 3927 50  0000 C CNN
+F 2 "" H 15200 4100 50  0001 C CNN
+F 3 "" H 15200 4100 50  0001 C CNN
+	1    15200 4100
+	-1   0    0    -1
+$EndComp
+Wire Wire Line
+	15200 4000 15200 4100
 $Comp
 L power:+3.3V #PWR0103
 U 1 1 5E926AF9
-P 15200 3300
-F 0 "#PWR0103" H 15200 3150 50  0001 C CNN
-F 1 "+3.3V" H 15215 3473 50  0000 C CNN
-F 2 "" H 15200 3300 50  0001 C CNN
-F 3 "" H 15200 3300 50  0001 C CNN
-	1    15200 3300
-	1    0    0    -1
-$EndComp
-$Comp
-L device:R_Small R14
+P 15200 2750
+F 0 "#PWR0103" H 15200 2600 50  0001 C CNN
+F 1 "+3.3V" H 15215 2923 50  0000 C CNN
+F 2 "" H 15200 2750 50  0001 C CNN
+F 3 "" H 15200 2750 50  0001 C CNN
+	1    15200 2750
+	1    0    0    -1
+$EndComp
+$Comp
+L HL2_MRF101-rescue:R_Small-device R14
 U 1 1 5EB97F20
-P 14350 4150
-F 0 "R14" V 14250 4150 50  0000 C CNN
-F 1 "JNC" V 14350 4150 39  0000 C CNN
-F 2 "Resistors_SMD:R_0805" H 14350 4150 50  0001 C CNN
-F 3 "~" H 14350 4150 50  0001 C CNN
-	1    14350 4150
+P 14350 3600
+F 0 "R14" V 14250 3600 50  0000 C CNN
+F 1 "JNC" V 14350 3600 39  0000 C CNN
+F 2 "Resistors_SMD:R_0805" H 14350 3600 50  0001 C CNN
+F 3 "~" H 14350 3600 50  0001 C CNN
+	1    14350 3600
 	0    1    1    0
 $EndComp
 $Comp
-L device:R_Small R35
+L HL2_MRF101-rescue:R_Small-device R35
 U 1 1 5EB9A462
-P 14350 4350
-F 0 "R35" V 14250 4350 50  0000 C CNN
-F 1 "JNC" V 14350 4350 39  0000 C CNN
-F 2 "Resistors_SMD:R_0805" H 14350 4350 50  0001 C CNN
-F 3 "~" H 14350 4350 50  0001 C CNN
-	1    14350 4350
+P 14350 3800
+F 0 "R35" V 14250 3800 50  0000 C CNN
+F 1 "JNC" V 14350 3800 39  0000 C CNN
+F 2 "Resistors_SMD:R_0805" H 14350 3800 50  0001 C CNN
+F 3 "~" H 14350 3800 50  0001 C CNN
+	1    14350 3800
 	0    1    1    0
 $EndComp
 $Comp
-L device:C_Small C83
+L HL2_MRF101-rescue:C_Small-device C83
 U 1 1 5ECD2378
-P 14600 4250
-F 0 "C83" H 14692 4296 50  0000 L CNN
-F 1 "DNI" H 14692 4205 50  0000 L CNN
-F 2 "Capacitors_SMD:C_0805" H 14600 4250 50  0001 C CNN
-F 3 "~" H 14600 4250 50  0001 C CNN
-	1    14600 4250
-	1    0    0    -1
-$EndComp
-Wire Wire Line
-	14600 4150 15000 4150
-Connection ~ 14600 4150
-Wire Wire Line
-	14600 4350 15000 4350
-Connection ~ 14600 4350
-Wire Wire Line
-	14450 4150 14600 4150
-Wire Wire Line
-	14450 4350 14600 4350
+P 14600 3700
+F 0 "C83" H 14692 3746 50  0000 L CNN
+F 1 "DNI" H 14692 3655 50  0000 L CNN
+F 2 "Capacitors_SMD:C_0805" H 14600 3700 50  0001 C CNN
+F 3 "~" H 14600 3700 50  0001 C CNN
+	1    14600 3700
+	1    0    0    -1
+$EndComp
+Wire Wire Line
+	14600 3600 15000 3600
+Connection ~ 14600 3600
+Wire Wire Line
+	14600 3800 15000 3800
+Connection ~ 14600 3800
+Wire Wire Line
+	14450 3600 14600 3600
+Wire Wire Line
+	14450 3800 14600 3800
 $Comp
 L HL2_MRF101-rescue:C_Small-Device C81
 U 1 1 5F1BB057
-P 15400 3700
-F 0 "C81" H 15492 3746 50  0000 L CNN
-F 1 "100n" H 15492 3655 50  0000 L CNN
-F 2 "Capacitors_SMD:C_0805" H 15400 3700 50  0001 C CNN
-F 3 "~" H 15400 3700 50  0001 C CNN
-	1    15400 3700
+P 15400 3150
+F 0 "C81" H 15492 3196 50  0000 L CNN
+F 1 "100n" H 15492 3105 50  0000 L CNN
+F 2 "Capacitors_SMD:C_0805" H 15400 3150 50  0001 C CNN
+F 3 "~" H 15400 3150 50  0001 C CNN
+	1    15400 3150
 	0    -1   -1   0
 $EndComp
@@
 L power:GND #PWR0110
 U 1 1 5F1BB4F8
-P 15550 3900
-F 0 "#PWR0110" H 15550 3650 50  0001 C CNN
-F 1 "GND" H 15555 3727 50  0000 C CNN
-F 2 "" H 15550 3900 50  0001 C CNN
-F 3 "" H 15550 3900 50  0001 C CNN
-	1    15550 3900
-	-1   0    0    -1
-$EndComp
-Wire Wire Line
-	15600 4250 15700 4250
-Text GLabel 15700 4250 2    50   Input ~ 0
+P 15550 3350
+F 0 "#PWR0110" H 15550 3100 50  0001 C CNN
+F 1 "GND" H 15555 3177 50  0000 C CNN
+F 2 "" H 15550 3350 50  0001 C CNN
+F 3 "" H 15550 3350 50  0001 C CNN
+	1    15550 3350
+	-1   0    0    -1
+$EndComp
+Wire Wire Line
+	15600 3700 15700 3700
+Text GLabel 15700 3700 2    50   Input ~ 0
 Vipa
 Wire Wire Line
-	15200 3700 15300 3700
-Wire Wire Line
-	15200 3700 15200 3950
-Wire Wire Line
-	15500 3700 15550 3700
-Wire Wire Line
-	15550 3700 15550 3900
-Wire Wire Line
-	15200 3600 15200 3700
-Connection ~ 15200 3700
+	15200 3150 15300 3150
+Wire Wire Line
+	15200 3150 15200 3400
+Wire Wire Line
+	15500 3150 15550 3150
+Wire Wire Line
+	15550 3150 15550 3350
+Wire Wire Line
+	15200 3050 15200 3150
+Connection ~ 15200 3150
 Wire Wire Line
 	8700 1400 8700 1700
@@
 Connection ~ 15550 1650
 $Comp
-L device:Ferrite_Bead_Small FB4
+L HL2_MRF101-rescue:Ferrite_Bead_Small-device FB4
 U 1 1 60A352B3
 P 15550 1250
@@
 Connection ~ 10650 10250
 $Comp
-L device:Ferrite_Bead_Small FB6
+L HL2_MRF101-rescue:Ferrite_Bead_Small-device FB6
 U 1 1 61A6DC40
-P 15200 3500
-F 0 "FB6" H 15100 3454 50  0000 R CNN
-F 1 "FB" H 15100 3545 50  0000 R CNN
-F 2 "Inductors_SMD:L_0805" V 15130 3500 50  0001 C CNN
-F 3 "~" H 15200 3500 50  0001 C CNN
-	1    15200 3500
+P 15200 2950
+F 0 "FB6" H 15100 2904 50  0000 R CNN
+F 1 "FB" H 15100 2995 50  0000 R CNN
+F 2 "Inductors_SMD:L_0805" V 15130 2950 50  0001 C CNN
+F 3 "~" H 15200 2950 50  0001 C CNN
+	1    15200 2950
 	1    0    0    1
 $EndComp
 Wire Wire Line
-	15200 3300 15200 3400
-$Comp
-L device:Ferrite_Bead_Small FB8
+	15200 2750 15200 2850
+$Comp
+L HL2_MRF101-rescue:Ferrite_Bead_Small-device FB8
 U 1 1 61B0B2C2
 P 15400 7850
@@
 	15400 7650 15400 7750
 $Comp
-L device:Ferrite_Bead_Small FB5
+L HL2_MRF101-rescue:Ferrite_Bead_Small-device FB5
 U 1 1 61BA94AF
 P 11950 1450
@@
 $EndComp
 $Comp
-L device:Ferrite_Bead_Small FB7
+L HL2_MRF101-rescue:Ferrite_Bead_Small-device FB7
 U 1 1 624EB2B1
 P 9250 3550
@@
 Connection ~ 9550 4350
 Connection ~ 9250 3750
-Text Notes 14450 4100 0    50   ~ 0
+Text Notes 14450 3550 0    50   ~ 0
 4A => 144mV
-Text Notes 15300 4750 0    50   ~ 0
+Text Notes 15300 4200 0    50   ~ 0
 Gain 20V/V\n4A => 2.88V
 $Comp
-L device:R_Small R34
+L HL2_MRF101-rescue:R_Small-device R34
 U 1 1 6355C858
-P 14000 4250
-F 0 "R34" H 13941 4204 50  0000 R CNN
-F 1 "0.036" H 13941 4295 50  0000 R CNN
-F 2 "Resistors_SMD:R_0612" H 14000 4250 50  0001 C CNN
-F 3 "~" H 14000 4250 50  0001 C CNN
-	1    14000 4250
+P 14000 3700
+F 0 "R34" H 13941 3654 50  0000 R CNN
+F 1 "0.036" H 13941 3745 50  0000 R CNN
+F 2 "Resistors_SMD:R_0612" H 14000 3700 50  0001 C CNN
+F 3 "~" H 14000 3700 50  0001 C CNN
+	1    14000 3700
 	1    0    0    1
 $EndComp
 Wire Wire Line
-	14000 4150 14250 4150
-Wire Wire Line
-	14000 4350 14250 4350
-Wire Wire Line
-	14000 4350 14000 4650
-Connection ~ 14000 4350
-Wire Wire Line
-	14000 3950 14000 4150
-Connection ~ 14000 4150
+	14000 3600 14250 3600
+Wire Wire Line
+	14000 3800 14250 3800
 Text GLabel 8250 1500 2    50   Input ~ 0
 Fan_Ctrl
@@
 Wire Wire Line
 	10100 1400 11550 1400
+Wire Wire Line
+	13550 3950 14000 3950
+Wire Wire Line
+	14000 3950 14000 3800
+Connection ~ 14000 3800
+Wire Wire Line
+	14000 3950 14000 4650
+Connection ~ 14000 3950
+Wire Wire Line
+	14000 3600 14000 2750
+Connection ~ 14000 3600
 $EndSCHEMATC

Commit message: Added ferrites, fan control
Added ferrite beads to relays
Added PWM fan control via DB1 on HL2
Parts:
- removed Q3: NSS60601MZ4, Package_TO_SOT_SMD:SOT-223-3_TabPin2, symbol HL2_MRF101-rescue:Q_NPN_BCE-Device
- removed R16, R17: 0, Resistor_SMD:R_0805_2012Metric, symbol HL2_MRF101-rescue:R_Small-Device
- removed R37: 10k, Resistor_SMD:R_0805_2012Metric, symbol HL2_MRF101-rescue:R_Small-Device
- added C84, C85: 1u, Capacitor_SMD:C_0805_2012Metric, symbol device:C_Small
- added D6: 1N4148W, Diode_SMD:D_SOD-123, symbol diode:1N4148W
- added FB10, FB11, FB12, FB13, FB14, FB15, FB16, FB17, FB18, FB9: FB, Inductor_SMD:L_0805_2012Metric, symbol device:Ferrite_Bead_Small
- added FB19: FB, Inductor_SMD:L_0805_2012Metric, symbol HL2_MRF101-rescue:Ferrite_Bead_Small-Device
- added J10: DB1, Pin_Headers:Pin_Header_Straight_1x06_Pitch2.54mm, symbol conn:Conn_01x06
- added Q3: IRLML6402, TO_SOT_Packages_SMD:SOT-23, symbol device:Q_PMOS_GSD
- added Q4: DTC144E, TO_SOT_Packages_SMD:SOT-23, symbol transistors:DTC144E
- added R16: 10k, Resistor_SMD:R_0805_2012Metric, symbol device:R_Small
- added R17: 1k, Resistor_SMD:R_0805_2012Metric, symbol device:R_Small
- added R36, R37, R38: TBD, Resistor_SMD:R_0805_2012Metric, symbol device:R_Small
- added TP2: P8, TestPoint:TestPoint_Pad_D1.5mm, symbol HL2_MRF101-rescue:TestPoint-Connector
- C78, C79, C80, C81, C82, C83: footprint Capacitors_SMD:C_0805 -> Capacitor_SMD:C_0805_2012Metric
- FB4, FB5, FB6, FB7, FB8: footprint Inductors_SMD:L_0805 -> Inductor_SMD:L_0805_2012Metric
- J3, J4: footprint n2adr:BNCEDGE -> n2adr:U.FL_Hirose_U.FL-R-SMT-1_Vertical
- R14, R35: footprint Resistors_SMD:R_0805 -> Resistor_SMD:R_0805_2012Metric
- R32: value 47k -> 100k
- R34: footprint Resistors_SMD:R_0612 -> Resistor_SMD:R_0612_1632Metric
- U6: footprint Housings_SSOP:MSOP-8_3x3mm_Pitch0.65mm -> Package_SO:MSOP-8_3x3mm_P0.65mm
- U7: footprint TO_SOT_Packages_SMD:SOT-23-5 -> Package_TO_SOT_SMD:SOT-23-5
Connections:
- net +12V: now also Q3.2 (S), R16.1; no longer J8.1 (Pin_1)
- net Band1: now also FB10.1, FB9.2; no longer C1.2, C38.2, K1.8, K6.8
- net Band2: now also FB11.2, FB12.1; no longer C2.2, C39.2, K2.8, K7.8
- net Band3: now also FB13.2, FB14.1; no longer C3.2, C40.2, K3.8, K8.8
- net Band4: now also FB15.2, FB16.1; no longer C4.2, C41.2, K4.8, K9.8
- net Band5: now also FB17.2, FB18.1; no longer C42.2, C5.2, K10.8, K5.8
- net Band7: now also FB19.2; no longer C64.2, K13.8
- net FWD_DET: now also J2.19 (Pin_19)
- net GND: now also J8.2 (Pin_2), C84.1, C85.1, D6.2 (A), J10.6 (Pin_6), Q4.2 (E), R37.1, R38.1
- net RFL_DET: now also J2.20 (Pin_20)
- net at J3.1 (In): now also R36.1, R38.2; no longer J2.6 (Pin_6)
- net Fan_Ctrl: no longer names the net of U3.19 (GP7)
- net Fan_Ctrl: now also TP2.1
- new net: C38.2, FB10.2, K6.8
- new net: C39.2, FB12.2, K7.8
- new net: C40.2, FB14.2, K8.8
- new net: C41.2, FB16.2, K9.8
- new net: C42.2, FB18.2, K10.8
- new net: C1.2, FB9.1, K1.8
- new net: C5.2, FB17.1, K5.8
- new net: C4.2, FB15.1, K4.8
- new net: C3.2, FB13.1, K3.8
- new net: C2.2, FB11.1, K2.8
- new net: J2.6 (Pin_6), R36.2, R37.2
- new net: C64.2, FB19.1, K13.8
- new net: C85.2, D6.1 (K), J8.1 (Pin_1), Q3.3 (D)
- new net: J10.1 (Pin_1), Q4.1 (B)
- new net: Q4.3 (C), R17.2
- new net: C84.2, Q3.1 (G), R16.2, R17.1
- no-connect marks 5 -> 9
Other:
- note added: "15-10 m"
- note added: "DB1 Pins 4-14"
- note added: "Set to 5k\nSet for 100mA\n=> Vipa = 72mV\n\nBias voltage ranges\nfrom 1 to 3.3 V"
- note removed: "15/12/10 m"
- note removed: "Set to 10k\nSet for 100mA\n=> Vipa = 72mV"
- moved on the sheet: C43, C44, C45, C46, C47, C48, C49, C50, C51, C52, C53, C61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
